File: kicad/vtbt.kicad_sch (KiCad schematic)
At the start: 33 parts, among them J1 955016449, Q1 MMBT4401, Q2 MMBT4401, Q3 MMBT4401, U1 ESP32-C3-DevKitM-1, U2 LT1032CSW-PBF, U3 MAX3183EEUK+T

Commit message: Reroute for rollover-wired modular cable
Phone handset cables are commonly available and use rollover-wiring.
Connections:
- net +12V: now also J1.2; no longer J1.3
- net GND: now also J1.3; no longer J1.2
- net RS_423_RX: now also J1.4; no longer J1.1
- net RS_423_TX: now also J1.1; no longer J1.4
